File: bkm10rduino.kicad_pcb (KiCad board)
At the start: 2 copper layers, 83.8 x 55.9 mm, 13 parts, among them SW1 SW_MEC_5E_copy, SW2 SW_MEC_5E_copy, SW3 SW_MEC_5E_copy, SW4 SW_MEC_5E_copy, SW5 SW_MEC_5E_copy, U1 TLL_TO_RS485

Commit message: update kicad layout
Parts:
- moved R5 0.71 mm to (164.1, 96.5)
Routing:
- net /5v: track 82.2 -> 0.00 mm
- net /g1: track 63.8 -> 0.40 mm, vias 0 -> 5
- net Net-(R5-Pad1): track 6.35 -> 7.06 mm
- added copper zone on In2.Cu, net /5v
- added copper zone on B.Cu, net /g1
- removed copper zone on F.Cu, net /g1
Other:
- copper layers 2 -> 4
Changed lines of the file:
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@@
     (thickness 1.6)
     (drawings 4)
-    (tracks 121)
+    (tracks 100)
     (zones 0)
     (modules 13)
@@
   (layers
     (0 F.Cu signal)
-    (31 B.Cu signal)
-    (32 B.Adhes user)
-    (33 F.Adhes user)
-    (34 B.Paste user)
-    (35 F.Paste user)
+    (1 In1.Cu signal)
+    (2 In2.Cu power)
+    (31 B.Cu power)
     (36 B.SilkS user)
     (37 F.SilkS user)
@@
   (module bkm10rduino:6_PIN_HEADER (layer F.Cu)
     (at 129.54 78.74 270)
-    (fp_text reference H1 (at 0 0.5 270) (layer F.SilkS)
+    (fp_text reference H1 (at 0 -8.89 270) (layer F.SilkS)
       (effects (font (size 1 1) (thickness 0.15)))
     )
@@
     (descr "Arduino UNO R3, http://www.mouser.com/pdfdocs/Gravitech_Arduino_Nano3_0.pdf")
     (tags "Arduino UNO R3")
-    (fp_text reference A1 (at 1.27 3.81 -180) (layer B.SilkS)
+    (fp_text reference A1 (at -2.54 0 -180) (layer B.SilkS)
       (effects (font (size 1 1) (thickness 0.15)) (justify mirror))
     )
@@
   )
   (module Resistor_SMD:R_1210_3225Metric_Pad1.30x2.65mm_HandSolder (layer F.Cu)
-    (at 164.82 96.52 180)
+    (at 164.11 96.52 180)
     (descr "Resistor SMD 1210 (3225 Metric), square (rectangular) end terminal, IPC_7351 nominal with elongated pad for handsoldering. (Body size source: IPC-SM-782 page 72, https://www.pcb-3d.com/wordpress/wp-content/uploads/ipc-sm-782a_amendment_1_and_2.pdf), generated with kicad-footprint-generator")
     (tags "resistor handsolder")
@@
   (gr_line (start 130.81 104.14) (end 130.81 48.26) (layer Edge.Cuts) (width 0.1))
   (gr_line (start 214.63 104.14) (end 130.81 104.14) (layer Edge.Cuts) (width 0.1))
+  (via (at 205.74 59.69) (size 0.8) (drill 0.4) (layers F.Cu B.Cu) (net 37))
+  (via (at 205.74 73.66) (size 0.8) (drill 0.4) (layers F.Cu B.Cu) (net 37))
   (segment (start 135.89 56.598001) (end 132.631999 56.598001) (width 0.25) (layer F.Cu) (net 11))
   (segment (start 132.631999 56.598001) (end 132.08 57.15) (width 0.25) (layer F.Cu) (net 11))
@@
   (segment (start 202.92 73.66) (end 202.92 75.21) (width 0.25) (layer F.Cu) (net 22))
   (segment (start 153.67 88.9) (end 153.67 92.71) (width 0.25) (layer F.Cu) (net 23))
-  (segment (start 166.37 96.52) (end 172.72 96.52) (width 0.25) (layer F.Cu) (net 24))
+  (segment (start 172.72 96.52) (end 165.66 96.52) (width 0.25) (layer F.Cu) (net 24))
   (segment (start 189.23 69.85) (end 189.23 76.2) (width 0.25) (layer F.Cu) (net 26))
   (segment (start 189.23 76.2) (end 186.69 78.74) (width 0.25) (layer F.Cu) (net 26))
@@
   (segment (start 191.31999 61.41001) (end 191.31999 67.76001) (width 0.25) (layer F.Cu) (net 26))
   (segment (start 200.66 52.07) (end 191.31999 61.41001) (width 0.25) (layer F.Cu) (net 26))
-  (segment (start 199.39 73.66) (end 199.39 74.93) (width 0.25) (layer F.Cu) (net 27))
-  (segment (start 199.39 74.93) (end 196.85 77.47) (width 0.25) (layer F.Cu) (net 27))
-  (segment (start 196.85 85.09) (end 199.39 87.63) (width 0.25) (layer F.Cu) (net 27))
-  (segment (start 196.85 77.47) (end 196.85 85.09) (width 0.25) (layer F.Cu) (net 27))
-  (segment (start 199.39 87.63) (end 196.85 87.63) (width 0.25) (layer F.Cu) (net 27))
-  (segment (start 186.69 97.79) (end 182.88 97.79) (width 0.25) (layer F.Cu) (net 27))
-  (segment (start 196.85 87.63) (end 186.69 97.79) (width 0.25) (layer F.Cu) (net 27))
-  (segment (start 199.39 59.69) (end 199.39 60.96) (width 0.25) (layer F.Cu) (net 27))
-  (segment (start 199.39 60.96) (end 198.12 62.23) (width 0.25) (layer F.Cu) (net 27))
-  (segment (start 198.12 72.39) (end 199.39 73.66) (width 0.25) (layer F.Cu) (net 27))
-  (segment (start 198.12 62.23) (end 198.12 72.39) (width 0.25) (layer F.Cu) (net 27))
-  (segment (start 182.88 99.06) (end 182.88 97.79) (width 0.25) (layer F.Cu) (net 27))
-  (segment (start 182.88 100.33) (end 182.88 99.06) (width 0.25) (layer F.Cu) (net 27))
-  (segment (start 181.61 96.52) (end 182.88 97.79) (width 0.25) (layer F.Cu) (net 27))
-  (segment (start 177.8 96.52) (end 181.61 96.52) (width 0.25) (layer F.Cu) (net 27))
-  (segment (start 170.18 88.9) (end 158.75 88.9) (width 0.25) (layer F.Cu) (net 27))
-  (segment (start 177.8 96.52) (end 170.18 88.9) (width 0.25) (layer F.Cu) (net 27))
+  (segment (start 177.8 96.52) (end 177.8 96.52) (width 0.25) (layer F.Cu) (net 27))
   (segment (start 193.04 52.07) (end 193.04 53.34) (width 0.25) (layer F.Cu) (net 28))
   (segment (start 193.04 53.34) (end 190.5 55.88) (width 0.25) (layer F.Cu) (net 28))
@@
   (segment (start 135.89 83.82) (end 135.89 64.218001) (width 0.25) (layer F.Cu) (net 38))
   (segment (start 133.35 86.36) (end 135.89 83.82) (width 0.25) (layer F.Cu) (net 38))
-  (segment (start 184.294999 101.455001) (end 185.42 100.33) (width 0.25) (layer F.Cu) (net 37))
-  (segment (start 154.38 96.52) (end 153.67 95.81) (width 0.25) (layer F.Cu) (net 37))
-  (segment (start 163.27 96.52) (end 154.38 96.52) (width 0.25) (layer F.Cu) (net 37))
-  (segment (start 168.205001 101.455001) (end 170.035001 101.455001) (width 0.25) (layer F.Cu) (net 37))
-  (segment (start 163.27 96.52) (end 168.205001 101.455001) (width 0.25) (layer F.Cu) (net 37))
-  (segment (start 170.035001 101.455001) (end 184.294999 101.455001) (width 0.25) (layer F.Cu) (net 37))
-  (segment (start 168.765001 101.455001) (end 170.035001 101.455001) (width 0.25) (layer F.Cu) (net 37))
-  (segment (start 188.41001 97.33999) (end 199.84001 97.33999) (width 0.25) (layer F.Cu) (net 37))
-  (segment (start 185.42 100.33) (end 188.41001 97.33999) (width 0.25) (layer F.Cu) (net 37))
-  (segment (start 199.84001 97.33999) (end 205.74 91.44) (width 0.25) (layer F.Cu) (net 37))
-  (segment (start 205.74 87.91) (end 206.02 87.63) (width 0.25) (layer F.Cu) (net 37))
-  (segment (start 205.74 91.44) (end 205.74 87.91) (width 0.25) (layer F.Cu) (net 37))
+  (segment (start 205.74 87.91) (end 205.88 87.77) (width 0.25) (layer F.Cu) (net 37))
+  (via (at 162.56 96.52) (size 0.8) (drill 0.4) (layers F.Cu B.Cu) (net 37))
+  (via (at 153.67 96.165) (size 0.8) (drill 0.4) (layers F.Cu B.Cu) (net 37))
+  (segment (start 205.88 87.77) (end 206.02 87.63) (width 0.25) (layer F.Cu) (net 37))
+  (via (at 205.88 87.77) (size 0.8) (drill 0.4) (layers F.Cu B.Cu) (net 37))
   (segment (start 185.934981 102.355019) (end 149.345019 102.355019) (width 0.25) (layer F.Cu) (net 38))
   (segment (start 187.96 100.33) (end 185.934981 102.355019) (width 0.25) (layer F.Cu) (net 38))
@@
   (segment (start 134.437001 75.112999) (end 134.437001 66.493411) (width 0.25) (layer F.Cu) (net 46))
   (segment (start 133.35 76.2) (end 134.437001 75.112999) (width 0.25) (layer F.Cu) (net 46))
-  (zone (net 37) (net_name /g1) (layer F.Cu) (hatch edge 0.508)
-    (connect_pads (clearance 0.508))
+  (zone (net 37) (net_name /g1) (layer B.Cu) (hatch edge 0.508)
+    (connect_pads yes (clearance 0.508))
     (min_thickness 0.254)
-    (fill yes (arc_segments 32) (thermal_gap 0.508) (thermal_bridge_width 0.508))
+    (fill yes (arc_segments 32) (thermal_gap 0.508) (thermal_bridge_width 0.508) (smoothing fillet) (radius 5))
     (polygon
       (pts
-        (xy 209.55 91.44) (xy 205.74 91.44) (xy 205.74 57.15) (xy 209.55 57.15)
+        (xy 214.63 104.14) (xy 130.81 104.14) (xy 130.81 48.26) (xy 214.63 48.26)
       )
     )
+  )
+  (zone (net 27) (net_name /5v) (layer In2.Cu) (hatch edge 0.508)
+    (connect_pads yes (clearance 0.508))
+    (min_thickness 0.254)
+    (fill yes (arc_segments 32) (thermal_gap 0.508) (thermal_bridge_width 0.508) (smoothing chamfer) (radius 5))
+    (polygon
+      (pts
+        (xy 214.63 104.14) (xy 130.81 104.14) (xy 130.81 48.26) (xy 214.63 48.26)
+      )
+    )
