File: kicad/All Controls/All Controls.sch (KiCad schematic (older format))
At the start: 2 parts

Commit message: fix beginneer mistakes on all controls
Connections:
- net labels added: GND
- net labels removed: GNDPWR
- wire segments 155 -> 139
Changed lines of the file:
@@
 L power:VCC #PWR0101
 U 1 1 619EE318
-P 4500 850
-F 0 "#PWR0101" H 4500 700 50  0001 C CNN
-F 1 "VCC" H 4515 1023 50  0000 C CNN
-F 2 "" H 4500 850 50  0001 C CNN
-F 3 "" H 4500 850 50  0001 C CNN
-	1    4500 850
+P 4500 1000
+F 0 "#PWR0101" H 4500 850 50  0001 C CNN
+F 1 "VCC" H 4515 1173 50  0000 C CNN
+F 2 "" H 4500 1000 50  0001 C CNN
+F 3 "" H 4500 1000 50  0001 C CNN
+	1    4500 1000
 	1    0    0    -1
 $EndComp
-$Comp
-L power:GNDPWR #PWR0102
-U 1 1 619EEE7B
-P 4850 850
-F 0 "#PWR0102" H 4850 650 50  0001 C CNN
-F 1 "GNDPWR" H 4854 696 50  0000 C CNN
-F 2 "" H 4850 800 50  0001 C CNN
-F 3 "" H 4850 800 50  0001 C CNN
-	1    4850 850
-	1    0    0    -1
-$EndComp
-Wire Wire Line
-	4500 850  4500 1000
-Wire Wire Line
-	4850 850  4650 850
-Wire Wire Line
-	4650 850  4650 1850
-Wire Wire Line
-	4650 1850 3000 1850
-Wire Wire Line
-	3000 1850 3000 3250
-Wire Wire Line
-	3000 3250 2700 3250
-Connection ~ 3000 1850
-Wire Wire Line
-	3000 1850 2650 1850
 Wire Wire Line
 	2700 3100 2900 3100
@@
 	850  3250 1150 3250
 Connection ~ 850  1700
-Wire Wire Line
-	4650 1850 4650 3250
-Wire Wire Line
-	4650 3250 6250 3250
-Connection ~ 4650 1850
 Wire Wire Line
 	4500 1000 6450 1000
@@
 Wire Wire Line
 	3400 2550 6850 2550
-Connection ~ 6250 3250
-Wire Wire Line
-	6250 3250 7350 3250
 $Sheet
 S 5250 6600 550  650
@@
 $EndSheet
 Wire Wire Line
-	6250 6850 5800 6850
-Wire Wire Line
-	5800 5900 6250 5900
-Connection ~ 6250 5900
-Wire Wire Line
-	6250 5900 6250 6850
-Wire Wire Line
-	5800 4950 6250 4950
-Wire Wire Line
-	6250 3250 6250 4050
-Connection ~ 6250 4950
-Wire Wire Line
-	6250 4950 6250 5900
-Wire Wire Line
-	5800 4050 6250 4050
-Connection ~ 6250 4050
-Wire Wire Line
-	6250 4050 6250 4950
-Wire Wire Line
 	6450 1000 6450 3950
 Wire Wire Line
@@
 	7850 2350 8450 2350
 Wire Wire Line
-	8450 2350 8450 6950
-Wire Wire Line
-	8450 6950 5800 6950
+	8450 2350 8450 6200
 Wire Wire Line
 	7850 2250 8550 2250
 Wire Wire Line
-	8550 2250 8550 7050
-Wire Wire Line
-	8550 7050 5800 7050
+	8550 2250 8550 6300
 NoConn ~ 7850 1650
 NoConn ~ 7850 1750
@@
 $EndComp
 Wire Wire Line
-	4650 3250 4200 3250
-Wire Wire Line
-	4200 3250 4200 4050
-Connection ~ 4650 3250
-Wire Wire Line
 	6450 5500 4200 5500
 Wire Wire Line
@@
 NoConn ~ 3800 4750
 NoConn ~ 3800 4450
+$Comp
+L power:GND #PWR0102
+U 1 1 6176B8F6
+P 2650 1850
+F 0 "#PWR0102" H 2650 1600 50  0001 C CNN
+F 1 "GND" V 2655 1722 50  0000 R CNN
+F 2 "" H 2650 1850 50  0001 C CNN
+F 3 "" H 2650 1850 50  0001 C CNN
+	1    2650 1850
+	0    -1   -1   0
+$EndComp
+$Comp
+L power:GND #PWR0103
+U 1 1 6176C95D
+P 2700 3250
+F 0 "#PWR0103" H 2700 3000 50  0001 C CNN
+F 1 "GND" V 2705 3122 50  0000 R CNN
+F 2 "" H 2700 3250 50  0001 C CNN
+F 3 "" H 2700 3250 50  0001 C CNN
+	1    2700 3250
+	0    -1   -1   0
+$EndComp
+$Comp
+L power:GND #PWR0104
+U 1 1 6176D341
+P 5800 5900
+F 0 "#PWR0104" H 5800 5650 50  0001 C CNN
+F 1 "GND" V 5805 5772 50  0000 R CNN
+F 2 "" H 5800 5900 50  0001 C CNN
+F 3 "" H 5800 5900 50  0001 C CNN
+	1    5800 5900
+	0    -1   -1   0
+$EndComp
+$Comp
+L power:GND #PWR0105
+U 1 1 6176E9D4
+P 5800 4950
+F 0 "#PWR0105" H 5800 4700 50  0001 C CNN
+F 1 "GND" V 5805 4822 50  0000 R CNN
+F 2 "" H 5800 4950 50  0001 C CNN
+F 3 "" H 5800 4950 50  0001 C CNN
+	1    5800 4950
+	0    -1   -1   0
+$EndComp
+$Comp
+L power:GND #PWR0106
+U 1 1 6176F137
+P 5800 4050
+F 0 "#PWR0106" H 5800 3800 50  0001 C CNN
+F 1 "GND" V 5805 3922 50  0000 R CNN
+F 2 "" H 5800 4050 50  0001 C CNN
+F 3 "" H 5800 4050 50  0001 C CNN
+	1    5800 4050
+	0    -1   -1   0
+$EndComp
+$Comp
+L power:GND #PWR0107
+U 1 1 6176F6CA
+P 5800 6850
+F 0 "#PWR0107" H 5800 6600 50  0001 C CNN
+F 1 "GND" V 5805 6722 50  0000 R CNN
+F 2 "" H 5800 6850 50  0001 C CNN
+F 3 "" H 5800 6850 50  0001 C CNN
+	1    5800 6850
+	0    -1   -1   0
+$EndComp
+$Comp
+L power:GND #PWR0108
+U 1 1 61770393
+P 7350 3250
+F 0 "#PWR0108" H 7350 3000 50  0001 C CNN
+F 1 "GND" H 7355 3077 50  0000 C CNN
+F 2 "" H 7350 3250 50  0001 C CNN
+F 3 "" H 7350 3250 50  0001 C CNN
+	1    7350 3250
+	1    0    0    -1
+$EndComp
+$Comp
+L power:GND #PWR0109
+U 1 1 6177171C
+P 4200 4050
+F 0 "#PWR0109" H 4200 3800 50  0001 C CNN
+F 1 "GND" H 4205 3877 50  0000 C CNN
+F 2 "" H 4200 4050 50  0001 C CNN
+F 3 "" H 4200 4050 50  0001 C CNN
+	1    4200 4050
+	-1   0    0    1
+$EndComp
+Wire Wire Line
+	6800 6950 6800 6200
+Wire Wire Line
+	6800 6200 8450 6200
+Wire Wire Line
+	6800 6950 5800 6950
+Wire Wire Line
+	8550 6300 6900 6300
+Wire Wire Line
+	6900 6300 6900 7050
+Wire Wire Line
+	6900 7050 5800 7050
 $EndSCHEMATC
