File: kicad/All Controls/OtherControls.sch (KiCad schematic (older format))
At the start: 28 parts, among them SW17 SW_SPST_LED, SW18 SW_SPST_LED, SW19 SW_SPST_LED, SW20 SW_SPST_LED, SW21 SW_SPST_LED, SW22 SW_SPST_LED, SW23 SW_SPST_LED, SW24 SW_SPST_LED, SW25 SW_SPST_LED, SW26 SW_SPST_LED

Commit message: fix beginneer mistakes on all controls
Connections:
- net GND: now also R17.1, R18.1, R19.1, R20.1, R21.1, R22.1, R23.1, R24.1, R25.1, R26.1, R27.1, R28.1, SW17.3 (K), SW18.3 (K), SW19.3 (K), SW20.3 (K), SW21.3 (K), SW22.3 (K), SW23.3 (K), SW24.3 (K), SW25.3 (K), SW26.3 (K); no longer Degauss1.2 (B), Power1.2 (B), SW17.2, SW18.2, SW19.2, SW20.2, SW21.2, SW22.2, SW23.2, SW24.2, SW25.2, SW26.2
- net VCC: now also Degauss1.2 (B), Power1.2 (B), SW17.2, SW18.2, SW19.2, SW20.2, SW21.2, SW22.2, SW23.2, SW24.2, SW25.2, SW26.2; no longer PISO3.11 (D0), PISO3.12 (D1), PISO3.13 (D2), PISO3.14 (D3), PISO3.3 (D4), PISO3.4 (D5), PISO3.5 (D6), PISO3.6 (D7), PISO4.11 (D0), PISO4.12 (D1), PISO4.13 (D2), PISO4.14 (D3), R17.2, R18.2, R19.2, R20.2, R21.2, R22.2, R23.2, R24.2, R25.2, R26.2, R27.2, R28.2, SW17.3 (K), SW18.3 (K), SW19.3 (K), SW20.3 (K), SW21.3 (K), SW22.3 (K), SW23.3 (K), SW24.3 (K), SW25.3 (K), SW26.3 (K)
- net at SW17.1: now also PISO3.6 (D7), R17.2; no longer R17.1
- net at SW18.1: now also PISO3.5 (D6), R18.2; no longer R18.1
- net at SW19.1: now also PISO3.4 (D5), R19.2; no longer R19.1
- net at SW20.1: now also PISO3.3 (D4), R20.2; no longer R20.1
- net at SW21.1: now also PISO3.14 (D3), R21.2; no longer R21.1
- net at SW22.1: now also PISO3.13 (D2), R22.2; no longer R22.1
- net at SW23.1: now also PISO3.12 (D1), R23.2; no longer R23.1
- net at SW24.1: now also PISO3.11 (D0), R24.2; no longer R24.1
- net at SW25.1: now also PISO4.14 (D3), R25.2; no longer R25.1
- net at SW26.1: now also PISO4.13 (D2), R26.2; no longer R26.1
- net at Degauss1.1 (A): now also PISO4.11 (D0), R28.2; no longer R28.1
- net at Power1.1 (A): now also PISO4.12 (D1), R27.2; no longer R27.1
Other:
- moved on the sheet: R17, R18, R19, R20, R21, R22, R23, R24, R25, R26, R27, R28
